Commit message: Update drone urdf.urdf

File: urdf/drone urdf.urdf (robot description, URDF)
Before this commit: robot drone urdf, 3 links, 2 joints
Links:
- link base_link: geometry collision mesh filename=package://drone_urdf/meshes/base_link.STL; visual mesh filename=package://drone_urdf/meshes/base_link.STL
- link link 2: geometry collision mesh filename=package://drone_urdf/meshes/link 2.STL; visual mesh filename=package://drone_urdf/meshes/link 2.STL
- link link1: geometry collision mesh filename=package://drone_urdf/meshes/link1.STL; visual mesh filename=package://drone_urdf/meshes/link1.STL
